File: hardware/PCB/SnapNodes-RP2_HAT_MediaLCD.kicad_pcb (KiCad board)
At the start: 4 copper layers, 40 x 40 mm, 89 parts, among them J1 USB_C, J2 LCD, J3 SPEAKER, J4 Conn_01x24_MountingPin, SW1 Left, SW2 Bottom, SW3 Right, SW4 Top, SW5 Center, U1 AW9523B, U2 NS4150B, U3 LSM6DS3, U4 TMD37253M, U5 XC6206P182MR, U6 24C02Cx-x-SN, U7 SHT45, U8 BMP280

Commit message: all V2 PCBs done
Signed-off-by: Hanxiang Chen <jhxchen7@outlook.com>
Parts:
- removed C9: 1n, Capacitor_SMD:C_0603_1608Metric
- C2: moved to F.Cu
- moved C24 5.31 mm to (124.2, 106.1), turned to 180 degrees
- moved R18 4.97 mm to (107.1, 107.5), turned to 90 degrees
- moved JP1 3.40 mm to (108.2, 126.4)
- moved JP3 3.40 mm to (112.5, 126.4)
- moved JP2 3.40 mm to (110.3, 126.4)
- moved J3 3.00 mm to (110.2, 114.0)
- moved U6 1.83 mm to (130.6, 109.3), turned to 165 degrees
- moved C8 1.50 mm to (102.6, 120.8)
- moved C6 1.13 mm to (111.6, 120.0), turned to 180 degrees
- moved R22 1.06 mm to (126.5, 107.2), turned to 75 degrees
- moved R1 1.00 mm to (122.2, 107.9)
- moved C2 0.70 mm to (105.8, 130.8), turned to 0 degrees
- moved G*** 0.30 mm to (128.3, 138.0)
Routing:
- net /SPK+: track 5.37 -> 14.2 mm
- net LCD_BL: track 22.6 -> 16.4 mm
- net COLOR_INT: track 28.4 -> 33.7 mm
- net +3V3: track 69.7 -> 74.3 mm, vias 34 -> 33
- net Net-(JP3-A): track 2.51 -> 5.06 mm
- net GND: track 41.6 -> 39.3 mm, vias 113 -> 114
- net I2C_SCL: track 138.4 -> 136.7 mm
- net Net-(JP1-A): track 4.34 -> 2.60 mm
- net I2C_SDA: track 131.0 -> 130.2 mm
- net VBUS: track 41.8 -> 41.2 mm
Other:
- outline, holes or cut-outs redrawn
- board text added: "1 2"
- board text added: "23 24"
- board text added: "SnapNodes-RP2 Hat V2"
- board text removed: "SnapNode-RP2 HAT V2"
