File: hardware/PCB/SnapNodes-RP2_Core.kicad_pcb (KiCad board)
At the start: 4 copper layers, 40 x 40 mm, 130 parts, among them J1 P_Female, J2 P_Male, J20 Conn_01x24_MountingPin, J3 P_Female, J4 P_Male, J5 P_Female, J6 P_Male, J7 P_Female, J8 P_Male, J9 SWD, Q1 2N7002W, U1 RP2350_80QFN, U2 TPS62A01PDDC, U3 BQ24232RGT, U4 ESP-PSRAM64H, U6 W25Q128JVSIQ, U7 74AHC1G04, Y1 12M

Commit message: HAT V2 PCB done, minor fix for Core PCB
Signed-off-by: Hanxiang Chen <jhxchen7@outlook.com>
Parts:
- added D29: PESD5V0S1BA, Diode_SMD:D_SOD-523, B.Cu at (102.5, 116.3)
- added D30: PESD5V0S1BA, Diode_SMD:D_SOD-523, B.Cu at (114.8, 136.3)
- added D31: PESD5V0S1BA, Diode_SMD:D_SOD-523, B.Cu at (137.6, 124.4)
- added D32: PESD5V0S1BA, Diode_SMD:D_SOD-523, B.Cu at (123.7, 102.5)
- added D33: PESD3V3S1BA, Diode_SMD:D_SOD-523, F.Cu at (120.3, 133.8)
- added D34: PESD3V3S1BA, Diode_SMD:D_SOD-523, F.Cu at (121.1, 136.0)
- D17, D18, D19: moved to F.Cu
- moved D3 7.24 mm to (109.5, 113.4), turned to 0 degrees
- moved D26 4.44 mm to (118.9, 103.0), turned to 0 degrees
- moved D7 4.16 mm to (107.4, 115.7), turned to 0 degrees
- moved D6 3.86 mm to (107.0, 113.4), turned to 0 degrees
- moved D11 3.67 mm to (133.0, 131.2), turned to -90 degrees
- moved D25 2.95 mm to (125.5, 106.3)
- moved D23 2.90 mm to (130.6, 106.3)
- moved D24 2.85 mm to (128.1, 106.2)
- moved D28 2.56 mm to (112.0, 104.2), turned to -45 degrees
- moved D18 2.53 mm to (113.2, 134.4)
- moved D17 2.51 mm to (110.7, 134.4)
- moved D19 2.51 mm to (115.7, 134.4)
- moved D13 2.46 mm to (134.2, 125.2), turned to 90 degrees
- moved D27 2.30 mm to (114.3, 103.7), turned to -60 degrees
- moved D12 1.12 mm to (135.6, 128.5)
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Connections:
- D10 pad 1: Net-(D10-K) -> /PA.CB
- D11 pad 1: Net-(D11-K) -> /PC.CA
- D12 pad 1: Net-(D12-K) -> /PC.D0
- D13 pad 1: Net-(D13-K) -> /PC.D1
- D14 pad 1: Net-(D14-K) -> /PC.D2
- D15 pad 1: Net-(D15-K) -> /PC.D3
- D16 pad 1: Net-(D16-K) -> /PC.CB
- D17 pad 1: Net-(D17-K) -> /PB.CA
- D18 pad 1: Net-(D18-K) -> /PB.D0
- D19 pad 1: Net-(D19-K) -> /PB.D1
- D20 pad 1: Net-(D20-K) -> /PB.D2
- D21 pad 1: Net-(D21-K) -> /PB.D3
- D22 pad 1: Net-(D22-K) -> /PB.CB
- D23 pad 1: Net-(D23-K) -> /PD.CA
- D24 pad 1: Net-(D24-K) -> /PD.D0
- D25 pad 1: Net-(D25-K) -> /PD.D1
- D26 pad 1: Net-(D26-K) -> /PD.D2
- D27 pad 1: Net-(D27-K) -> /PD.D3
- D28 pad 1: Net-(D28-K) -> /PD.CB
- D3 pad 1: Net-(D3-K) -> /PA.CA
- D6 pad 1: Net-(D6-K) -> /PA.D0
- D7 pad 1: Net-(D7-K) -> /PA.D1
- D8 pad 1: Net-(D8-K) -> /PA.D2
- D9 pad 1: Net-(D9-K) -> /PA.D3
- J1 pad 2: Net-(D8-K) -> Net-(J1-Pin_2)
- J1 pad 3: Net-(D9-K) -> Net-(J1-Pin_3)
- J1 pad 4: Net-(D10-K) -> Net-(J1-Pin_4)
- J2 pad 2: Net-(D3-K) -> Net-(J2-Pin_2)
- J2 pad 3: Net-(D6-K) -> Net-(J2-Pin_3)
- J2 pad 4: Net-(D7-K) -> Net-(J2-Pin_4)
- J3 pad 2: Net-(D20-K) -> Net-(J3-Pin_2)
- J3 pad 3: Net-(D21-K) -> Net-(J3-Pin_3)
- J3 pad 4: Net-(D22-K) -> Net-(J3-Pin_4)
- J4 pad 2: Net-(D17-K) -> Net-(J4-Pin_2)
- J4 pad 3: Net-(D18-K) -> Net-(J4-Pin_3)
- J4 pad 4: Net-(D19-K) -> Net-(J4-Pin_4)
- J5 pad 2: Net-(D14-K) -> Net-(J5-Pin_2)
- J5 pad 3: Net-(D15-K) -> Net-(J5-Pin_3)
- J5 pad 4: Net-(D16-K) -> Net-(J5-Pin_4)
- J6 pad 2: Net-(D11-K) -> Net-(J6-Pin_2)
- J6 pad 3: Net-(D12-K) -> Net-(J6-Pin_3)
- J6 pad 4: Net-(D13-K) -> Net-(J6-Pin_4)
- J7 pad 2: Net-(D26-K) -> Net-(J7-Pin_2)
- J7 pad 3: Net-(D27-K) -> Net-(J7-Pin_3)
- J7 pad 4: Net-(D28-K) -> Net-(J7-Pin_4)
- J8 pad 2: Net-(D23-K) -> Net-(J8-Pin_2)
- J8 pad 3: Net-(D24-K) -> Net-(J8-Pin_3)
- J8 pad 4: Net-(D25-K) -> Net-(J8-Pin_4)
- R1 pad 1: Net-(D3-K) -> Net-(J2-Pin_2)
- R10 pad 1: Net-(D23-K) -> Net-(J8-Pin_2)
- R11 pad 1: Net-(D25-K) -> Net-(J8-Pin_4)
- R12 pad 1: Net-(D27-K) -> Net-(J7-Pin_3)
- R2 pad 1: Net-(D7-K) -> Net-(J2-Pin_4)
- R3 pad 1: Net-(D9-K) -> Net-(J1-Pin_3)
- R31 pad 1: Net-(D6-K) -> Net-(J2-Pin_3)
- R32 pad 1: Net-(D8-K) -> Net-(J1-Pin_2)
- R33 pad 1: Net-(D10-K) -> Net-(J1-Pin_4)
- R35 pad 1: Net-(D12-K) -> Net-(J6-Pin_3)
- R36 pad 1: Net-(D14-K) -> Net-(J5-Pin_2)
- R37 pad 1: Net-(D16-K) -> Net-(J5-Pin_4)
- R38 pad 1: Net-(D18-K) -> Net-(J4-Pin_3)
- R39 pad 1: Net-(D20-K) -> Net-(J3-Pin_2)
- R4 pad 1: Net-(D17-K) -> Net-(J4-Pin_2)
- R40 pad 1: Net-(D22-K) -> Net-(J3-Pin_4)
- R41 pad 1: Net-(D24-K) -> Net-(J8-Pin_3)
- R42 pad 1: Net-(D26-K) -> Net-(J7-Pin_2)
- R43 pad 1: Net-(D28-K) -> Net-(J7-Pin_4)
- R5 pad 1: Net-(D19-K) -> Net-(J4-Pin_4)
- R6 pad 1: Net-(D21-K) -> Net-(J3-Pin_3)
- R7 pad 1: Net-(D11-K) -> Net-(J6-Pin_2)
- R8 pad 1: Net-(D13-K) -> Net-(J6-Pin_4)
- R9 pad 1: Net-(D15-K) -> Net-(J5-Pin_3)
Routing:
- net Net-(J2-Pin_2): track 0.00 -> 5.83 mm
- net Net-(D3-K): track 5.83 -> 0.00 mm, vias 1 -> 0
- net Net-(D22-K): track 2.59 -> 0.00 mm
- net Net-(D21-K): track 2.59 -> 0.00 mm
- net Net-(D20-K): track 2.59 -> 0.00 mm
- net Net-(D16-K): track 2.59 -> 0.00 mm
- net Net-(D15-K): track 2.59 -> 0.00 mm
- net Net-(D14-K): track 2.59 -> 0.00 mm
- net Net-(D28-K): track 2.57 -> 0.00 mm
- net Net-(D9-K): track 2.39 -> 0.00 mm
- net Net-(D8-K): track 2.39 -> 0.00 mm
- net Net-(D10-K): track 2.39 -> 0.00 mm
- net Net-(D26-K): track 2.30 -> 0.00 mm
- net Net-(D27-K): track 2.00 -> 0.00 mm
- net VIN: track 33.5 -> 35.5 mm
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- added copper zone on B.Cu, net VIN
Other:
- board text added: "1 2"
- board text added: "23 24"

Commit message: all V2 PCBs done
Signed-off-by: Hanxiang Chen <jhxchen7@outlook.com>
Parts:
- C8: footprint Capacitor_SMD:C_0402_1005Metric -> Capacitor_SMD:C_0805_2012Metric
- moved BT1 1.41 mm to (109.3, 130.7)
- moved C8 0.69 mm to (129.2, 134.6)
- moved L2 0.30 mm to (132.3, 133.3)
Routing:
- net +BATT: track 47.1 -> 44.2 mm
- net GND: track 34.6 -> 35.3 mm, vias 126 -> 128
- net +3V3: vias 40 -> 39
Other:
- outline, holes or cut-outs redrawn
- board text added: "SnapNodes-RP2 Core V2"
- board text removed: "SnapNode-RP2 Core V2"

Commit message: changed LCSC P/N of 5V TVS, moved a MLCC that conflicts with FPC connector on core board
Signed-off-by: Hanxiang Chen <jhxchen7@outlook.com>
Parts:
- moved C7 2.23 mm to (131.3, 130.7), turned to -90 degrees
Routing:
- net GND: track 35.3 -> 36.7 mm
- added copper zone on F.Cu, net VBUS
Other:
- board text added: "SnapNodes-RP2 Core V2.1"
- board text added: "shBLOCK Jason Chen 2026.09"
- board text removed: "SnapNodes-RP2 Core V2"
- board text removed: "shBLOCK Jason Chen 2026.08"
