File: hardware/PCB/SnapNodes_Breakout.kicad_sch (KiCad schematic)
At the start: 24 parts, among them J1 P_Male, J2 P_Female, J3 Conn_01x08, J4 U.FL, J5 U.FL, J6 U.FL, J7 U.FL, J8 U.FL, J9 U.FL

Commit message: changed LCSC P/N of 5V TVS, moved a MLCC that conflicts with FPC connector on core board
Signed-off-by: Hanxiang Chen <jhxchen7@outlook.com>
Parts:
- D7: LCSC P/N C5158048 -> C314264
Changed lines of the file:
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@@
 			)
 		)
-		(property "LCSC P/N" "C5158048"
+		(property "LCSC P/N" "C314264"
 			(at 133.35 55.88 0)
 			(hide yes)
